File: hardware/PCB/Sensor_array/Sensor_array.kicad_sch (KiCad schematic)
At the start: 29 parts, among them J2 8x2 Sensor Connector, Q1 BSS214NW, U1 QRE1113GR, U10 QRE1113GR, U2 QRE1113GR, U3 QRE1113GR, U6 QRE1113GR, U7 QRE1113GR, U8 QRE1113GR, U9 QRE1113GR

Commit message: Flipped connector and added insightful silkscreen to sensor array
Connections:
- net S1: now also R6.2, U10.3; no longer R12.2, U1.3
- net S2: now also R7.2, U9.3; no longer R13.2, U2.3
- net S3: now also R9.2, U8.3; no longer R10.2, U3.3
- net S4: now also R8.2, U7.3; no longer R11.2, U6.3
- net S5: now also R11.2, U6.3; no longer R8.2, U7.3
- net S6: now also R10.2, U3.3; no longer R9.2, U8.3
- net S7: now also R13.2, U2.3; no longer R7.2, U9.3
- net S8: now also R12.2, U1.3; no longer R6.2, U10.3
Changed lines of the file:
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@@
 		)
 	)
-	(label "S1"
+	(label "S8"
 		(at 114.3 48.26 0)
 		(fields_autoplaced yes)
@@
 		)
 	)
-	(label "S2"
+	(label "S7"
 		(at 118.745 73.66 0)
 		(fields_autoplaced yes)
@@
 		)
 	)
-	(label "S7"
+	(label "S2"
 		(at 198.755 48.26 0)
 		(fields_autoplaced yes)
@@
 		)
 	)
-	(label "S3"
+	(label "S6"
 		(at 141.605 48.26 0)
 		(fields_autoplaced yes)
@@
 		)
 	)
-	(label "S5"
+	(label "S4"
 		(at 169.545 48.26 0)
 		(fields_autoplaced yes)
@@
 		)
 	)
-	(label "S6"
+	(label "S3"
 		(at 173.99 73.66 0)
 		(fields_autoplaced yes)
@@
 		)
 	)
-	(label "S8"
+	(label "S1"
 		(at 203.2 73.66 0)
 		(fields_autoplaced yes)
@@
 		)
 	)
-	(label "S4"
+	(label "S5"
 		(at 146.05 73.66 0)
 		(fields_autoplaced yes)
