File: hardware/PCB/Sensor_array/Sensor_array.kicad_pcb (KiCad board)
At the start: 2 copper layers, 80 x 16.5 mm, 29 parts, among them J2 8x2 Sensor Connector, Q1 BSS214NW, U1 QRE1113GR, U10 QRE1113GR, U2 QRE1113GR, U3 QRE1113GR, U6 QRE1113GR, U7 QRE1113GR, U8 QRE1113GR, U9 QRE1113GR

Commit message: Flipped connector and added insightful silkscreen to sensor array
Parts:
- C1, C2, J2, Q1, R14, R15, R5: moved to B.Cu
- moved R14 50.4 mm to (116.2, 88.0), turned to -90 degrees
- moved R15 48.1 mm to (118.2, 88.0), turned to -90 degrees
- moved Q1 45.9 mm to (116.2, 92.0), turned to 90 degrees
- moved R5 42.9 mm to (119.2, 91.9), turned to -90 degrees
- moved C1 25.6 mm to (127.5, 95.0), turned to 0 degrees
- moved C2 25.6 mm to (127.5, 93.0), turned to 0 degrees
- moved J2 17.8 mm to (148.9, 94.8)
Connections:
- R10 pad 2: /S3 -> /S6
- R11 pad 2: /S4 -> /S5
- R12 pad 2: /S1 -> /S8
- R13 pad 2: /S2 -> /S7
- R6 pad 2: /S8 -> /S1
- R7 pad 2: /S7 -> /S2
- R8 pad 2: /S5 -> /S4
- R9 pad 2: /S6 -> /S3
- U1 pad 3: /S1 -> /S8
- U10 pad 3: /S8 -> /S1
- U2 pad 3: /S2 -> /S7
- U3 pad 3: /S3 -> /S6
- U6 pad 3: /S4 -> /S5
- U7 pad 3: /S5 -> /S4
- U8 pad 3: /S6 -> /S3
- U9 pad 3: /S7 -> /S2
Routing:
- net VCC: track 36.0 -> 12.1 mm, vias 0 -> 2
- net Net-(U10-K): track 81.6 -> 70.3 mm, vias 5 -> 4
- net /S7: track 23.5 -> 19.5 mm
- net /S2: track 19.4 -> 23.5 mm
- net /S6: track 16.0 -> 12.0 mm
- net /S3: track 12.0 -> 16.0 mm
- net /S8: track 31.0 -> 27.0 mm
- net /S1: track 27.0 -> 30.9 mm
- net GND: track 14.9 -> 12.3 mm, vias 10 -> 8
- net /S4: track 6.64 -> 8.54 mm
- net /S5: track 8.58 -> 7.39 mm
- net /SENSOR_LED: track 17.2 -> 16.3 mm
Other:
- board text added: "EN"
- board text added: "S1"
- board text added: "S8"
- board text added: "VCC"

Commit message: Initial payload control board and connector layout
Other:
- board text added: "EGB220 A10"
Changed lines of the file:
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@@
 		)
 		(fp_text user "${REFERENCE}"
-			(at 0 0 360)
+			(at 0 0 0)
 			(layer "B.Fab")
 			(effects
@@
 		)
 	)
+	(gr_text "EGB220 A10"
+		(at 159.75 95.5 0)
+		(layer "F.SilkS")
+		(effects
+			(font
+				(size 1 1)
+				(thickness 0.1)
+			)
+			(justify left bottom)
+		)
+	)

Commit message: Finished PCBs for payload and turret
Changed lines of the file:
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@@
 	)
 	(segment
-		(start 172 84)
-		(end 174.1 84)
+		(start 174.1 84)
+		(end 172 84)
 		(width 0.3)
 		(layer "F.Cu")

Commit message: Final project commit
Other:
- board text removed: "EGB220 A10"
