File: hardware/PCB/payload_controlboard/payload_controlboard.kicad_pcb (KiCad board)
At the start: 2 copper layers, 65 x 45 mm, 13 parts, among them J1 Servo_X, J2 Servo_Y, J3 IR_Tracker, J4 Laser, J5 linefollower->payload

Commit message: payload v2
Parts:
- removed 100R: 100R, Resistor_THT:R_Axial_DIN0207_L6.3mm_D2.5mm_P10.16mm_Horizontal
- removed POWER: PWR, LED_THT:LED_D5.0mm
- removed RESET: SW_MEC_5E, Button_Switch_THT:SO4_222A-M-V-B_CTS
- removed Teensy 2.0: Teensy2.0_(C), Module:Teensy2.0
- added D1: PWR, LED_THT:LED_D5.0mm, F.Cu at (112.5, 107.5)
- added R1: 100R, Resistor_THT:R_Axial_DIN0207_L6.3mm_D2.5mm_P10.16mm_Horizontal, F.Cu at (113.5, 90.9)
- added SW1: RST, footprints:SO4_222A-M-V-B_CTS, F.Cu at (142.0, 112.7)
- added SW2: MODE, footprints:SO4_222A-M-V-B_CTS, F.Cu at (153.0, 112.8)
- added U2: Teensy2.0_(C), footprints:Teensy2.0, F.Cu at (127.5, 95.5)
Routing:
- net Net-(U2-PD4_ADC8_ICP1): track 0.00 -> 31.2 mm
- net Net-(SW1-A): track 0.00 -> 14.8 mm
- net GND: track 1.50 -> 13.6 mm
- net Net-(U2-RST): track 10.6 -> 0.00 mm
